File: hardware/Opt101/Opt101.sch (KiCad schematic (older format))
At the start: 19 parts, among them J1 DIN_4, U1 OPT101, U3 UAF42

Commit message: Reorganized directories.
Parts:
- RV1: symbol POT -> POT-RESCUE-Opt101
Changed lines of the file:
@@
-EESchema Schematic File Version 2
-LIBS:Opt101-rescue
+EESchema Schematic File Version 3
 LIBS:power
-LIBS:device
-LIBS:conn
-LIBS:linear
-LIBS:regul
-LIBS:74xx
-LIBS:cmos4000
-LIBS:adc-dac
-LIBS:memory
-LIBS:xilinx
-LIBS:microcontrollers
-LIBS:dsp
-LIBS:microchip
-LIBS:analog_switches
-LIBS:motorola
-LIBS:texas
-LIBS:intel
-LIBS:audio
-LIBS:interface
-LIBS:digital-audio
-LIBS:philips
-LIBS:display
-LIBS:cypress
-LIBS:siliconi
-LIBS:contrib
-LIBS:valves
 LIBS:light_sensor_boards
 LIBS:components
+LIBS:Opt101-rescue
 LIBS:Opt101-cache
-EELAYER 25 0
+EELAYER 26 0
 EELAYER END
 $Descr A 11000 8500
@@
 NoConn ~ 6400 3050
 $Comp
-L POT RV1
+L POT-RESCUE-Opt101 RV1
 U 1 1 49FF78C5
 P 7600 2800
